File: xc6slx16-devboard/xc6slx16-devboard.kicad_pcb (KiCad board)
At the start: 4 copper layers, 67.6 x 30 mm, 30 parts, among them IC2 M25P80-VMN6P, IC3 25MHz, J1 SODIMM-200_Split, J3 Conn_02x05_Odd_Even, U1 XC6SLX16-FTG256, U2 K4X1G163PE

Commit message: devboard
Parts:
- added C1: 1u, Capacitor_SMD:C_0603_1608Metric, F.Cu at (168.4, 29.4)
- added C10: 10u, Capacitor_SMD:C_0603_1608Metric, F.Cu at (172.4, 26.1)
- added C11: 8.2p, Capacitor_SMD:C_0402_1005Metric, F.Cu at (176.2, 31.6)
- added C12: 6.8p, Capacitor_SMD:C_0402_1005Metric, F.Cu at (183.9, 23.6)
- added C13: 33p, Capacitor_SMD:C_0402_1005Metric, F.Cu at (176.2, 29.6)
- added C14: 10u, Capacitor_SMD:C_0603_1608Metric, F.Cu at (172.4, 28.7)
- added C15: 10u, Capacitor_SMD:C_0603_1608Metric, F.Cu at (185.5, 15.2)
- added C16: 4.7u, Capacitor_SMD:C_0805_2012Metric, F.Cu at (152.8, 31.2)
- added C17: 4.7u, Capacitor_SMD:C_0805_2012Metric, F.Cu at (170.8, 16.2)
- added C2: 1u, Capacitor_SMD:C_0603_1608Metric, F.Cu at (179.7, 19.4)
- added C3: 1u, Capacitor_SMD:C_0603_1608Metric, F.Cu at (174.8, 18.9)
- added C30: 1u, Capacitor_SMD:C_0603_1608Metric_Pad1.08x0.95mm_HandSolder, F.Cu at (136.4, -7.02)
- added C31: 1u, Capacitor_SMD:C_0603_1608Metric_Pad1.08x0.95mm_HandSolder, F.Cu at (136.4, -4.51)
- added C32: 22p, Capacitor_SMD:C_0402_1005Metric, F.Cu at (181.7, 25.6)
- added C33: 1u, Capacitor_SMD:C_0603_1608Metric_Pad1.08x0.95mm_HandSolder, F.Cu at (140.8, -7.02)
- added C34: 4.7u, Capacitor_SMD:C_0805_2012Metric, F.Cu at (170.6, 19.2)
- added C35: 22p, Capacitor_SMD:C_0402_1005Metric, F.Cu at (185.0, 21.4)
- added C36: 100n, Capacitor_SMD:C_01005_0402Metric, F.Cu at (159.6, 165.7)
- added C37: 100n, Capacitor_SMD:C_01005_0402Metric, F.Cu at (149.8, 176.3)
- added C4: 4.7u, Capacitor_SMD:C_0603_1608Metric, F.Cu at (164.0, 31.1)
- added C5: 4.7u, Capacitor_SMD:C_0603_1608Metric, F.Cu at (168.4, 26.9)
- added C6: 1u, Capacitor_SMD:C_0603_1608Metric, F.Cu at (175.7, 21.4)
- added C7: 10u, Capacitor_SMD:C_0603_1608Metric, F.Cu at (178.9, 16.9)
- added C8: 100n, Capacitor_SMD:C_0402_1005Metric, F.Cu at (181.7, 27.6)
- added C9: 10u, Capacitor_SMD:C_0603_1608Metric, F.Cu at (185.5, 12.7)
- added D1: Diode_Schottky, dsi_shield:SOD3715X145N, F.Cu at (153.6, 28.1)
- added D2: Diode_Schottky, dsi_shield:SOD3715X145N, F.Cu at (160.9, 23.5)
- added D3: Diode_Schottky, dsi_shield:SOD3715X145N, F.Cu at (165.3, 19.3)
- added D4: Diode_Schottky, dsi_shield:SOD3715X145N, F.Cu at (171.6, 13.0)
- added D6: PRTR5V0U2X, Package_TO_SOT_SMD:SOT-143, F.Cu at (148.6, 164.7)
- added D7: PRTR5V0U2X, Package_TO_SOT_SMD:SOT-143, F.Cu at (137.2, 174.9)
- added D8: IP4292CZ10, dsi_shield:SOT1176-1, F.Cu at (156.6, 164.0)
- added D9: IP4292CZ10, dsi_shield:SOT1176-1, F.Cu at (151.4, 168.6)
- added IC1: LM26480, Package_DFN_QFN:WQFN-24-1EP_4x4mm_P0.5mm_EP2.6x2.6mm, F.Cu at (165.4, 14.5)
- added IC4: SOT95P275X110-5N, mybays:SOT95P275X110-5N, F.Cu at (166.6, 23.3)
- added IC5: SOT95P275X110-5N, mybays:SOT95P275X110-5N, F.Cu at (159.4, 28.7)
- added J2: Conn_02x15_Odd_Even, Connector_PinHeader_2.54mm:PinHeader_2x15_P2.54mm_Vertical, F.Cu at (70.6, 67.1)
- added L1: 2.2uH, dsi_shield:IND_PANASONIC_ELLVEG, F.Cu at (180.3, 13.5)
- added L2: 2.2uH, dsi_shield:IND_PANASONIC_ELLVEG, F.Cu at (170.5, 22.8)
- added L3: 4.7uH, dsi_shield:IND_PANASONIC_ELLVEG, F.Cu at (163.2, 27.7)
- added L4: 4.7uH, dsi_shield:IND_PANASONIC_ELLVEG, F.Cu at (175.9, 13.5)
- added P1: USB_C_Plug, Connector_USB:USB_C_Receptacle_HRO_TYPE-C-31-M-12, F.Cu at (139.0, 11.9)
- added Q1: 2N7002, Package_TO_SOT_SMD:SOT-23, F.Cu at (146.4, 174.9)
- added Q2: 2N7002, Package_TO_SOT_SMD:SOT-23, F.Cu at (153.4, 164.7)
- added Q3: Q_BSS84, Package_TO_SOT_SMD:SOT-23, F.Cu at (148.2, 169.2)
- added Q4: 2N7002, Package_TO_SOT_SMD:SOT-23, F.Cu at (142.0, 174.9)
- added R10: 560k, Resistor_SMD:R_0402_1005Metric, F.Cu at (186.1, 17.4)
- added R11: 178k, Resistor_SMD:R_0402_1005Metric, F.Cu at (175.9, 27.7)
- added R12: 100k, Resistor_SMD:R_0402_1005Metric, F.Cu at (183.2, 19.4)
- added R13: 0, Resistor_SMD:R_0402_1005Metric, F.Cu at (183.2, 17.4)
- added R14: 0, Resistor_SMD:R_0402_1005Metric, F.Cu at (178.1, 23.7)
- added R15: 100k, Resistor_SMD:R_0402_1005Metric, F.Cu at (175.2, 23.7)
- added R16: 100k, Resistor_SMD:R_0402_1005Metric, F.Cu at (167.5, 31.6)
- added R17: 27k, Resistor_SMD:R_0402_1005Metric, F.Cu at (179.2, 21.6)
- added R18: 100k, Resistor_SMD:R_0402_1005Metric, F.Cu at (175.9, 25.7)
- added R19: 27k, Resistor_SMD:R_0402_1005Metric, F.Cu at (170.4, 31.6)
- added R2: 180, Resistor_SMD:R_0402_1005Metric, F.Cu at (196.1, 12.4)
- added R20: 3.3k, Resistor_SMD:R_0402_1005Metric, F.Cu at (157.1, 165.9)
- added R21: 3.3k, Resistor_SMD:R_0402_1005Metric, F.Cu at (155.7, 167.9)
- added R22: 1M, Resistor_SMD:R_0402_1005Metric, F.Cu at (151.9, 170.4)
- added R23: 3.3k, Resistor_SMD:R_0402_1005Metric, F.Cu at (150.1, 172.5)
- added R24: 3.3k, Resistor_SMD:R_0402_1005Metric, F.Cu at (150.1, 174.5)
- added R25: 3.3k, Resistor_SMD:R_0402_1005Metric, F.Cu at (153.0, 172.4)
- added R3: 220, Resistor_SMD:R_0402_1005Metric, F.Cu at (193.2, 12.4)
- added R35: 3.3k, Resistor_SMD:R_0402_1005Metric, F.Cu at (154.8, 170.4)
- added R37: 1k, Resistor_SMD:R_0402_1005Metric, F.Cu at (158.6, 167.9)
- added R38: 3.3k, Resistor_SMD:R_0402_1005Metric, F.Cu at (153.0, 174.4)
- added R39: 3.3k, Resistor_SMD:R_0402_1005Metric, F.Cu at (155.9, 172.4)
- added R4: 100k, Resistor_SMD:R_0402_1005Metric, F.Cu at (178.8, 25.7)
- added R40: 160, Resistor_SMD:R_0402_1005Metric, F.Cu at (97.6, 82.4)
- added R41: 160, Resistor_SMD:R_0402_1005Metric, F.Cu at (86.0, 82.4)
- added R42: 22, Resistor_SMD:R_0402_1005Metric, F.Cu at (88.9, 82.4)
- added R43: 22, Resistor_SMD:R_0402_1005Metric, F.Cu at (91.8, 82.4)
- added R44: 51, Resistor_SMD:R_0402_1005Metric, F.Cu at (94.7, 82.4)
- added R45: 51, Resistor_SMD:R_0402_1005Metric, F.Cu at (103.4, 86.3)
- added R46: 160, Resistor_SMD:R_0402_1005Metric, F.Cu at (100.5, 82.4)
- added R47: 160, Resistor_SMD:R_0402_1005Metric, F.Cu at (103.4, 82.4)
- added R48: 22, Resistor_SMD:R_0402_1005Metric, F.Cu at (106.3, 82.4)
- added R49: 22, Resistor_SMD:R_0402_1005Metric, F.Cu at (109.2, 82.4)
- added R5: 280k, Resistor_SMD:R_0402_1005Metric, F.Cu at (181.0, 23.6)
- added R50: 160, Resistor_SMD:R_0402_1005Metric, F.Cu at (112.2, 82.4)
- added R51: 160, Resistor_SMD:R_0402_1005Metric, F.Cu at (115.1, 82.4)
- added R52: 22, Resistor_SMD:R_0402_1005Metric, F.Cu at (118.0, 82.4)
- added R53: 22, Resistor_SMD:R_0402_1005Metric, F.Cu at (86.0, 84.3)
- added R54: 51, Resistor_SMD:R_0402_1005Metric, F.Cu at (88.9, 84.3)
- added R55: 51, Resistor_SMD:R_0402_1005Metric, F.Cu at (91.8, 84.3)
- added R56: 51, Resistor_SMD:R_0402_1005Metric, F.Cu at (94.7, 84.3)
- added R57: 51, Resistor_SMD:R_0402_1005Metric, F.Cu at (97.6, 84.3)
- added R58: 160, Resistor_SMD:R_0402_1005Metric, F.Cu at (100.5, 84.3)
- added R59: 160, Resistor_SMD:R_0402_1005Metric, F.Cu at (103.4, 84.3)
- added R6: 750k, Resistor_SMD:R_0402_1005Metric, F.Cu at (173.3, 30.9)
- added R60: 22, Resistor_SMD:R_0402_1005Metric, F.Cu at (106.3, 84.3)
- added R61: 22, Resistor_SMD:R_0402_1005Metric, F.Cu at (109.2, 84.3)
- added R62: 160, Resistor_SMD:R_0402_1005Metric, F.Cu at (112.2, 84.3)
- added R63: 160, Resistor_SMD:R_0402_1005Metric, F.Cu at (115.1, 84.3)
- added R64: 22, Resistor_SMD:R_0402_1005Metric, F.Cu at (86.0, 86.3)
- added R65: 22, Resistor_SMD:R_0402_1005Metric, F.Cu at (88.9, 86.3)
- added R66: 51, Resistor_SMD:R_0402_1005Metric, F.Cu at (91.8, 86.3)
- added R67: 51, Resistor_SMD:R_0402_1005Metric, F.Cu at (94.7, 86.3)
- added R68: 51, Resistor_SMD:R_0402_1005Metric, F.Cu at (97.6, 86.3)
- added R69: 51, Resistor_SMD:R_0402_1005Metric, F.Cu at (100.5, 86.3)
- added R7: 200k, Resistor_SMD:R_0402_1005Metric, F.Cu at (186.1, 19.4)
- added R8: 187k, Resistor_SMD:R_0402_1005Metric, F.Cu at (178.8, 27.7)
- added R9: 464k, Resistor_SMD:R_0402_1005Metric, F.Cu at (182.1, 21.6)
- added U3: CH340E, Package_SO:MSOP-10-1EP_3x3mm_P0.5mm_EP1.68x1.88mm_ThermalVias, F.Cu at (154.2, 24.1)
- J1: value SODIMM-200_Split -> 10118241-001RLF; footprint sodimm:SODIMM_DDR3_EDGE -> 10118241001RLF:10118241001RLF
- moved J1 49.3 mm to (114.2, 147.2)
- moved J3 13.8 mm to (169.4, 65.6)
Connections:
- net Net-(J1-Pad13) renamed HDMI_CEC
- net Net-(U1-PadM6) renamed /Sheet5FC7E9FD/DBG_O2
- net Net-(U1-PadN6) renamed /Sheet5FC7E9FD/DBG_O1
- net Net-(U1-PadR3) renamed /Sheet5FC7E9FD/DBG_O0
- net Net-(U1-PadT4) renamed /Sheet5FC7E9FD/DBG_O3
- net Net-(U1-PadT5) renamed /Sheet5FC7E9FD/VID_RESET_N
- IC3 pad 3: CLK_25MHZ -> /Sheet5FC7E9FD/CLK_25MHZ
- J1 pad 1: Net-(J1-Pad1) -> /Sheet6028F128/TMDS2_P
- J1 pad 10: Net-(J1-Pad10) -> /Sheet6028F128/TMDS_CLK_P
- J1 pad 11: Net-(J1-Pad11) -> GND
- J1 pad 12: Net-(J1-Pad12) -> /Sheet6028F128/TMDS_CLK_N
- J1 pad 15: Net-(J1-Pad15) -> HDMI_SCL
- J1 pad 16: Net-(J1-Pad16) -> HDMI_SDA
- J1 pad 17: Net-(J1-Pad17) -> GND
- J1 pad 18: Net-(J1-Pad18) -> HDMI_P5V
- J1 pad 19: Net-(J1-Pad19) -> HDMI_HPD
- J1 pad 2: Net-(J1-Pad2) -> GND
- J1 pad 3: Net-(J1-Pad3) -> /Sheet6028F128/TMDS2_N
- J1 pad 4: Net-(J1-Pad4) -> /Sheet6028F128/TMDS1_P
- J1 pad 5: Net-(J1-Pad5) -> GND
- J1 pad 6: Net-(J1-Pad6) -> /Sheet6028F128/TMDS1_N
- J1 pad 7: Net-(J1-Pad7) -> /Sheet6028F128/TMDS0_P
- J1 pad 8: Net-(J1-Pad8) -> GND
- J1 pad 9: Net-(J1-Pad9) -> /Sheet6028F128/TMDS0_N
- U1 pad A4: /Sheet5FC7E9FD/HPD_NOTIFY -> Net-(U1-PadA4)
- U1 pad A5: /Sheet5FC7E9FD/TMDS0_N -> Net-(U1-PadA5)
- U1 pad A6: /Sheet5FC7E9FD/TMDS2_N -> Net-(U1-PadA6)
- U1 pad A7: /Sheet5FC7E9FD/SDA -> Net-(U1-PadA7)
- U1 pad A8: /Sheet5FC7E9FD/DBG_RX -> Net-(U1-PadA8)
- U1 pad B1: Net-(U1-PadB1) -> DSI_HS_CLK_N
- U1 pad B5: /Sheet5FC7E9FD/TMDS0_P -> Net-(U1-PadB5)
- U1 pad B6: /Sheet5FC7E9FD/TMDS2_P -> Net-(U1-PadB6)
- U1 pad B8: /Sheet5FC7E9FD/DBG_TX -> Net-(U1-PadB8)
- U1 pad C1: Net-(U1-PadC1) -> DSI_HS_CLK_P
- U1 pad C2: Net-(U1-PadC2) -> DSI_LP_CLK_N
- U1 pad C3: Net-(U1-PadC3) -> DSI_LP_CLK_P
- U1 pad C4: /Sheet5FC7E9FD/BL_DIM -> Net-(U1-PadC4)
- U1 pad C5: /Sheet5FC7E9FD/TMDS1_N -> Net-(U1-PadC5)
- U1 pad C7: /Sheet5FC7E9FD/SCL -> Net-(U1-PadC7)
- U1 pad D5: /Sheet5FC7E9FD/TMDS1_P -> Net-(U1-PadD5)
- U1 pad D6: /Sheet5FC7E9FD/HPD_EN -> Net-(U1-PadD6)
- U1 pad E1: Net-(U1-PadE1) -> DSI_LP_0_N
- U1 pad E2: Net-(U1-PadE2) -> DSI_LP_0_P
- U1 pad E6: /Sheet5FC7E9FD/TMDS_CLK_N -> Net-(U1-PadE6)
- U1 pad F1: Net-(U1-PadF1) -> DSI_HS_0_N
- U1 pad F2: Net-(U1-PadF2) -> DSI_HS_0_P
- U1 pad F7: /Sheet5FC7E9FD/TMDS_CLK_P -> Net-(U1-PadF7)
- U1 pad G1: Net-(U1-PadG1) -> DSI_LP_1_N
- U1 pad G3: Net-(U1-PadG3) -> DSI_LP_1_P
- U1 pad H1: Net-(U1-PadH1) -> DSI_HS_1_N
- U1 pad H2: Net-(U1-PadH2) -> DSI_HS_1_P
- U1 pad J1: Net-(U1-PadJ1) -> DSI_LP_2_N
- U1 pad J3: Net-(U1-PadJ3) -> DSI_LP_2_P
- U1 pad K1: Net-(U1-PadK1) -> DSI_HS_2_N
- U1 pad K2: Net-(U1-PadK2) -> DSI_HS_2_P
- U1 pad L1: Net-(U1-PadL1) -> DSI_LP_3_N
- U1 pad L10: Net-(U1-PadL10) -> /Sheet5FC7E9FD/TMDS0_P
- U1 pad L3: Net-(U1-PadL3) -> DSI_LP_3_P
- U1 pad M1: Net-(U1-PadM1) -> DSI_HS_3_N
- U1 pad M10: Net-(U1-PadM10) -> /Sheet5FC7E9FD/TMDS0_N
- U1 pad M2: Net-(U1-PadM2) -> DSI_HS_3_P
- U1 pad M3: Net-(U1-PadM3) -> DSI_GPIO1
- U1 pad M4: Net-(U1-PadM4) -> DSI_GPIO0
- U1 pad M5: Net-(U1-PadM5) -> DSI_RESET_N
- U1 pad M9: Net-(U1-PadM9) -> /Sheet5FC7E9FD/TMDS2_P
- U1 pad N4: Net-(U1-PadN4) -> LCD_PWREN
- U1 pad N5: Net-(U1-PadN5) -> /Sheet5FC7E9FD/DBG_TX
- U1 pad N8: Net-(U1-PadN8) -> /Sheet5FC7E9FD/TMDS2_N
- U1 pad P5: Net-(U1-PadP5) -> /Sheet5FC7E9FD/DBG_RX
- U1 pad P6: Net-(U1-PadP6) -> /Sheet5FC7E9FD/HPD_NOTIFY
- U1 pad P8: Net-(U1-PadP8) -> /Sheet5FC7E9FD/TMDS_CLK_P
- U1 pad R5: Net-(U1-PadR5) -> /Sheet5FC7E9FD/BL_DIM
- U1 pad R7: Net-(U1-PadR7) -> /Sheet5FC7E9FD/SCL
- U1 pad R9: Net-(U1-PadR9) -> /Sheet5FC7E9FD/TMDS1_P
- U1 pad T6: Net-(U1-PadT6) -> /Sheet5FC7E9FD/HPD_EN
- U1 pad T7: Net-(U1-PadT7) -> /Sheet5FC7E9FD/SDA
- U1 pad T8: Net-(U1-PadT8) -> /Sheet5FC7E9FD/TMDS_CLK_N
- U1 pad T9: Net-(U1-PadT9) -> /Sheet5FC7E9FD/TMDS1_N
Other:
- board outline removed

Commit message: 20201130
Parts:
- removed R13, R14: 0, Resistor_SMD:R_0402_1005Metric
- R50: renamed from R48; moved to B.Cu
- R51: renamed from R49; moved to B.Cu
- R52: renamed from R60; moved to B.Cu
- R53: renamed from R61; moved to B.Cu
- R54: renamed from R42; moved to B.Cu
- R55: renamed from R43; moved to B.Cu
- R56: renamed from R52; moved to B.Cu
- R57: renamed from R53; moved to B.Cu
- R58: renamed from R64; moved to B.Cu
- R59: renamed from R65; moved to B.Cu
- moved C31 109.0 mm to (111.7, 101.7), turned to 180 degrees
- moved C30 108.6 mm to (116.2, 99.7)
- moved R17 101.4 mm to (117.0, 101.7), turned to 90 degrees
- moved C32 101.3 mm to (114.9, 101.7), turned to 270 degrees
- moved D7 99.7 mm to (166.6, 79.7)
- moved D4 95.6 mm to (125.7, 96.9), turned to 270 degrees
- moved R15 94.1 mm to (123.4, 102.2)
- moved C34 93.5 mm to (125.7, 101.3), turned to 270 degrees
- moved IC4 90.8 mm to (120.0, 101.2)
- moved D2 90.7 mm to (111.7, 99.7)
- moved R16 87.0 mm to (115.9, 101.7), turned to 270 degrees
- moved L3 81.6 mm to (121.0, 97.6), turned to 180 degrees
- moved C35 80.2 mm to (113.8, 58.5), turned to 270 degrees
- moved C16 80.0 mm to (120.2, 104.3), turned to 180 degrees
- moved R2 79.3 mm to (130.3, 56.8)
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- renumbered R46 to R40, R47 to R41, R58 to R42, R59 to R43, R40 to R44, R41 to R45, R50 to R46, R51 to R47, R62 to R48, R63 to R49, R54 to R60, R55 to R61, R66 to R62, R67 to R63, R44 to R64, R45 to R65, R56 to R66, R57 to R67
Connections:
- C11 pad 2: +1V8 -> V_DDR
- C14 pad 1: +1V8 -> V_DDR
- C2 pad 1: +1V8 -> V_DDR
- D8 pad 1: /Sheet6028F128/TMDS1_N -> /Sheet5FC7E9FD/TMDS1_N
- D8 pad 10: /Sheet6028F128/TMDS1_N -> /Sheet5FC7E9FD/TMDS1_N
- D8 pad 2: /Sheet6028F128/TMDS1_P -> /Sheet5FC7E9FD/TMDS1_P
- D8 pad 4: /Sheet6028F128/TMDS2_N -> /Sheet5FC7E9FD/TMDS2_N
- D8 pad 5: /Sheet6028F128/TMDS2_P -> /Sheet5FC7E9FD/TMDS2_P
- D8 pad 6: /Sheet6028F128/TMDS2_P -> /Sheet5FC7E9FD/TMDS2_P
- D8 pad 7: /Sheet6028F128/TMDS2_N -> /Sheet5FC7E9FD/TMDS2_N
- D8 pad 9: /Sheet6028F128/TMDS1_P -> /Sheet5FC7E9FD/TMDS1_P
- D9 pad 1: /Sheet6028F128/TMDS_CLK_N -> /Sheet5FC7E9FD/TMDS_CLK_N
- D9 pad 10: /Sheet6028F128/TMDS_CLK_N -> /Sheet5FC7E9FD/TMDS_CLK_N
- D9 pad 2: /Sheet6028F128/TMDS_CLK_P -> /Sheet5FC7E9FD/TMDS_CLK_P
- D9 pad 4: /Sheet6028F128/TMDS0_N -> /Sheet5FC7E9FD/TMDS0_N
- D9 pad 5: /Sheet6028F128/TMDS0_P -> /Sheet5FC7E9FD/TMDS0_P
- D9 pad 6: /Sheet6028F128/TMDS0_P -> /Sheet5FC7E9FD/TMDS0_P
- D9 pad 7: /Sheet6028F128/TMDS0_N -> /Sheet5FC7E9FD/TMDS0_N
- D9 pad 9: /Sheet6028F128/TMDS_CLK_P -> /Sheet5FC7E9FD/TMDS_CLK_P
- IC1 pad 19: +1V8 -> V_DDR
- J1 pad 1: /Sheet6028F128/TMDS2_P -> /Sheet5FC7E9FD/TMDS2_P
- J1 pad 10: /Sheet6028F128/TMDS_CLK_P -> /Sheet5FC7E9FD/TMDS_CLK_P
- J1 pad 12: /Sheet6028F128/TMDS_CLK_N -> /Sheet5FC7E9FD/TMDS_CLK_N
- J1 pad 3: /Sheet6028F128/TMDS2_N -> /Sheet5FC7E9FD/TMDS2_N
- J1 pad 4: /Sheet6028F128/TMDS1_P -> /Sheet5FC7E9FD/TMDS1_P
- J1 pad 6: /Sheet6028F128/TMDS1_N -> /Sheet5FC7E9FD/TMDS1_N
- J1 pad 7: /Sheet6028F128/TMDS0_P -> /Sheet5FC7E9FD/TMDS0_P
- J1 pad 9: /Sheet6028F128/TMDS0_N -> /Sheet5FC7E9FD/TMDS0_N
- J2 pad 19: +1V8 -> V_DDR
- L1 pad 2: +1V8 -> V_DDR
- Q1 pad 3: /Sheet6028F128/SDA -> /Sheet5FC7E9FD/SDA
- Q2 pad 3: /Sheet6028F128/SCL -> /Sheet5FC7E9FD/SCL
- Q4 pad 1: /Sheet6028F128/HPD_EN -> /Sheet5FC7E9FD/HPD_EN
- R20 pad 2: /Sheet6028F128/HPD_NOTIFY -> /Sheet5FC7E9FD/HPD_NOTIFY
- R21 pad 1: /Sheet6028F128/HPD_NOTIFY -> /Sheet5FC7E9FD/HPD_NOTIFY
- R25 pad 2: /Sheet6028F128/SDA -> /Sheet5FC7E9FD/SDA
- R35 pad 2: /Sheet6028F128/SCL -> /Sheet5FC7E9FD/SCL
- R39 pad 1: /Sheet6028F128/HPD_EN -> /Sheet5FC7E9FD/HPD_EN
- R9 pad 1: +1V8 -> V_DDR
- U1 pad B1: DSI_HS_CLK_N -> DSI_HS_3_N
- U1 pad C1: DSI_HS_CLK_P -> DSI_HS_3_P
- U1 pad C2: DSI_LP_CLK_N -> DSI_LP_3_N
- U1 pad C3: DSI_LP_CLK_P -> DSI_LP_3_P
- U1 pad D1: Net-(U1-PadD1) -> DSI_LP_2_N
- U1 pad D15: +1V8 -> V_DDR
- U1 pad D2: +1V8 -> V_DDR
- U1 pad D3: Net-(U1-PadD3) -> DSI_LP_2_P
- U1 pad E1: DSI_LP_0_N -> DSI_HS_2_N
- U1 pad E2: DSI_LP_0_P -> DSI_HS_2_P
- U1 pad F1: DSI_HS_0_N -> DSI_HS_CLK_N
- U1 pad F2: DSI_HS_0_P -> DSI_HS_CLK_P
- U1 pad G1: DSI_LP_1_N -> DSI_LP_CLK_N
- U1 pad G13: +1V8 -> V_DDR
- U1 pad G3: DSI_LP_1_P -> DSI_LP_CLK_P
- U1 pad G4: +1V8 -> V_DDR
- U1 pad H1: DSI_HS_1_N -> Net-(U1-PadH1)
- U1 pad H2: DSI_HS_1_P -> Net-(U1-PadH2)
- U1 pad J1: DSI_LP_2_N -> Net-(U1-PadJ1)
- U1 pad J15: +1V8 -> V_DDR
- U1 pad J2: +1V8 -> V_DDR
- U1 pad J3: DSI_LP_2_P -> Net-(U1-PadJ3)
- U1 pad K1: DSI_HS_2_N -> DSI_HS_1_N
- U1 pad K13: +1V8 -> V_DDR
- U1 pad K2: DSI_HS_2_P -> DSI_HS_1_P
- U1 pad K4: +1V8 -> V_DDR
- U1 pad L1: DSI_LP_3_N -> DSI_LP_1_N
- U1 pad L10: /Sheet5FC7E9FD/TMDS0_P -> Net-(U1-PadL10)
- U1 pad L3: DSI_LP_3_P -> DSI_LP_1_P
- U1 pad M1: DSI_HS_3_N -> DSI_GPIO1
- U1 pad M10: /Sheet5FC7E9FD/TMDS0_N -> Net-(U1-PadM10)
- U1 pad M2: DSI_HS_3_P -> DSI_RESET_N
- U1 pad M3: DSI_GPIO1 -> Net-(U1-PadM3)
- U1 pad M4: DSI_GPIO0 -> Net-(U1-PadM4)
- U1 pad M5: DSI_RESET_N -> Net-(U1-PadM5)
- U1 pad N1: Net-(U1-PadN1) -> DSI_GPIO0
- U1 pad N15: +1V8 -> V_DDR
- U1 pad N2: +1V8 -> V_DDR
- U1 pad P1: Net-(U1-PadP1) -> DSI_LP_0_N
- U1 pad P2: Net-(U1-PadP2) -> DSI_LP_0_P
- U1 pad P8: /Sheet5FC7E9FD/TMDS_CLK_P -> Net-(U1-PadP8)
- U1 pad R1: Net-(U1-PadR1) -> DSI_HS_0_N
- U1 pad R13: +1V8 -> V_DDR
- U1 pad R2: Net-(U1-PadR2) -> DSI_HS_0_P
- U1 pad R5: /Sheet5FC7E9FD/BL_DIM -> /Sheet5FC7E9FD/TMDS_CLK_P
- U1 pad R7: /Sheet5FC7E9FD/SCL -> /Sheet5FC7E9FD/TMDS0_P
- U1 pad T5: /Sheet5FC7E9FD/VID_RESET_N -> /Sheet5FC7E9FD/TMDS_CLK_N
- U1 pad T7: /Sheet5FC7E9FD/SDA -> /Sheet5FC7E9FD/TMDS0_N
- U1 pad T8: /Sheet5FC7E9FD/TMDS_CLK_N -> Net-(U1-PadT8)
Routing:
- net LCD_BOOST_FB: track 0.00 -> 54.3 mm
- net DSI_RESET_N: track 0.00 -> 33.2 mm, vias 0 -> 1
- net DSI_GPIO0: track 0.00 -> 28.9 mm
- net DSI_GPIO1: track 0.00 -> 27.1 mm
- net DSI_L0_N: track 0.00 -> 17.4 mm, vias 0 -> 1
- net DSI_L3_P: track 0.00 -> 17.3 mm, vias 0 -> 1
- net DSI_L0_P: track 0.00 -> 17.0 mm, vias 0 -> 1
- net DSI_L3_N: track 0.00 -> 16.9 mm, vias 0 -> 1
- net Net-(C30-Pad1): track 0.00 -> 15.9 mm
- net DSI_L2_N: track 0.00 -> 14.2 mm, vias 0 -> 1
- net DSI_L1_P: track 0.00 -> 14.2 mm, vias 0 -> 1
- net DSI_L2_P: track 0.00 -> 13.3 mm, vias 0 -> 1
- net DSI_L1_N: track 0.00 -> 13.3 mm, vias 0 -> 1
- net LCD_BL_FB: track 0.00 -> 13.1 mm
- net DSI_CLK_N: track 0.00 -> 12.5 mm, vias 0 -> 1
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Other:
- board outline added: 75 x 70 mm
- net class 2 added: clearance 0.2032, trace_width 0.2032, via_dia 0.4, via_drill 0.2

Commit message: 20201204
Parts:
- added C38: C, Capacitor_SMD:C_0402_1005Metric_Pad0.74x0.62mm_HandSolder, F.Cu at (123.7, 89.4)
- added R13: 4.7k, Resistor_SMD:R_0402_1005Metric, F.Cu at (159.2, 72.5)
- added R14: 100, Resistor_SMD:R_0402_1005Metric, B.Cu at (147.5, 68.4)
- added R70: 100k, Resistor_SMD:R_0402_1005Metric, F.Cu at (125.7, 52.0)
- added SW1: SW_Push, mybays_connector:turtlekey, F.Cu at (123.8, 87.1)
- C10, C14, C15, C9: footprint Capacitor_SMD:C_0603_1608Metric -> Capacitor_SMD:C_0805_2012Metric_Pad1.18x1.45mm_HandSolder
- C16, C17: footprint Capacitor_SMD:C_0805_2012Metric -> Capacitor_SMD:C_0603_1608Metric_Pad1.08x0.95mm_HandSolder
- C20: footprint Capacitor_SMD:C_0402_1005Metric -> Capacitor_SMD:C_0603_1608Metric_Pad1.08x0.95mm_HandSolder
- C21, C22, C23, C27, D6, D7, R1, R36: moved to B.Cu
- C34: footprint Capacitor_SMD:C_0805_2012Metric -> Capacitor_SMD:C_0805_2012Metric_Pad1.18x1.45mm_HandSolder
- C36, C37: footprint Capacitor_SMD:C_01005_0402Metric -> Capacitor_SMD:C_0402_1005Metric_Pad0.74x0.62mm_HandSolder
- moved D5 79.9 mm to (145.1, 97.0)
- moved R29 77.7 mm to (146.0, 98.9), turned to 270 degrees
- moved R30 75.4 mm to (144.2, 99.0), turned to 90 degrees
- moved R32 74.0 mm to (135.6, 100.3), turned to 270 degrees
- moved C19 73.6 mm to (145.1, 100.7), turned to 180 degrees
- moved R36 71.1 mm to (136.3, 77.5), turned to 90 degrees
- moved R26 66.6 mm to (128.1, 87.1), turned to 180 degrees
- moved R33 65.3 mm to (139.1, 91.1), turned to 180 degrees
- moved R34 64.4 mm to (131.6, 91.7)
- moved R27 63.4 mm to (146.6, 83.9)
- moved C24 62.0 mm to (154.4, 81.9)
- moved C20 62.0 mm to (160.2, 77.4), turned to 270 degrees
- moved R31 61.0 mm to (144.4, 84.0)
- moved C26 59.5 mm to (156.4, 81.9), turned to 180 degrees
- moved C22 58.5 mm to (149.0, 77.2), turned to 90 degrees
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Connections:
- net /Sheet5FC7E9FD/DBG_O0 renamed Net-(U1-PadR3)
- net /Sheet5FC7E9FD/DBG_O1 renamed Net-(U1-PadN6)
- net /Sheet5FC7E9FD/DBG_O2 renamed Net-(U1-PadM6)
- net /Sheet5FC7E9FD/DBG_O3 renamed Net-(U1-PadT4)
- net Net-(R36-Pad1) renamed /Sheet5FC7E9FD/FPGA_M1
- net Net-(U1-PadA6) renamed DBG_O2
- net Net-(U1-PadB6) renamed DBG_O3
- net Net-(U1-PadE6) renamed DBG_O0
- net Net-(U1-PadF7) renamed DBG_O1
- IC5 pad 4: +3V3 -> /Sheet5FC7E9FD/BL_DIM
- R28 pad 2: GND -> +3V3
- R34 pad 1: CPU_RST -> +3V3
- U1 pad A9: Net-(U1-PadA9) -> LCD_PWREN
- U1 pad C6: Net-(U1-PadC6) -> /Sheet5FC7E9FD/DBG_RX
- U1 pad C9: Net-(U1-PadC9) -> /Sheet5FC7E9FD/BL_DIM
- U1 pad D6: Net-(U1-PadD6) -> /Sheet6028E9E5/DBG_RX
- U1 pad N14: Net-(U1-PadN14) -> /Sheet5FC7E9FD/SDRAM_DQS0
- U1 pad N5: /Sheet5FC7E9FD/DBG_TX -> /Sheet5FC7E9FD/SCL
- U1 pad P5: /Sheet5FC7E9FD/DBG_RX -> /Sheet5FC7E9FD/SDA
- U1 pad R14: /Sheet5FC7E9FD/SDRAM_DQS0 -> /Sheet5FC7E9FD/SDRAM_DQS1
- U1 pad T15: /Sheet5FC7E9FD/SDRAM_DQS1 -> Net-(U1-PadT15)
- U3 pad 8: /Sheet6028E9E5/DBG_TX -> /Sheet5FC7E9FD/DBG_RX
Routing:
- net /Sheet5FC7E9FD/HPD_NOTIFY: track 0.00 -> 57.0 mm, vias 0 -> 2
- net /Sheet5FC7E9FD/HPD_EN: track 0.00 -> 50.2 mm, vias 0 -> 2
- net /Sheet5FC7E9FD/TMDS_CLK_P: track 0.00 -> 45.1 mm, vias 0 -> 2
- net /Sheet5FC7E9FD/TMDS_CLK_N: track 0.00 -> 45.0 mm, vias 0 -> 2
- net LCD_BOOST_FB: track 54.3 -> 10.7 mm
- net /Sheet5FC7E9FD/SDA: track 0.00 -> 42.8 mm, vias 0 -> 2
- net HDMI_P5V: track 0.00 -> 40.3 mm, vias 0 -> 3
- net /Sheet5FC7E9FD/TMDS1_P: track 0.00 -> 39.0 mm, vias 0 -> 2
- net /Sheet5FC7E9FD/TMDS0_P: track 0.00 -> 38.7 mm
- net /Sheet5FC7E9FD/TMDS1_N: track 0.00 -> 38.5 mm, vias 0 -> 2
- net /Sheet5FC7E9FD/TMDS0_N: track 0.00 -> 38.2 mm
- net /Sheet5FC7E9FD/TMDS2_N: track 0.00 -> 38.0 mm, vias 0 -> 2
- net /Sheet5FC7E9FD/TMDS2_P: track 0.00 -> 37.5 mm, vias 0 -> 2
- net /Sheet5FC7E9FD/QSPI_DQ1: track 0.71 -> 38.2 mm, vias 1 -> 6
- net /Sheet5FC7E9FD/QSPI_DQ2: track 0.71 -> 36.9 mm, vias 1 -> 6
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Other:
- board size 75 x 70 mm -> 75 x 65 mm

Commit message: 20201205
Parts:
- removed P1: USB_C_Plug, Connector_USB:USB_C_Receptacle_HRO_TYPE-C-31-M-12
- added D11: LED, LED_SMD:LED_0603_1608Metric_Pad1.05x0.95mm_HandSolder, F.Cu at (172.0, 74.6)
- added J4: Conn_02x15_Odd_Even, Connector_PinHeader_2.54mm:PinHeader_2x15_P2.54mm_Vertical, F.Cu at (118.0, 45.7)
- added J5: USB_C, mybays_connector:USB_C, F.Cu at (170.7, 59.9)
- added R72: 1k, Resistor_SMD:R_0402_1005Metric, F.Cu at (169.0, 74.6)
- moved J3 26.4 mm to (111.6, 46.9), turned to 0 degrees
- moved C8 26.3 mm to (140.4, 59.4), turned to 180 degrees
- moved C7 25.0 mm to (160.1, 46.9)
- moved R70 7.53 mm to (122.1, 58.6), turned to 90 degrees
- moved R2 5.64 mm to (128.4, 51.5)
- moved R3 5.64 mm to (128.4, 53.1)
- moved C18 5.64 mm to (124.1, 55.6)
- moved IC3 5.64 mm to (124.1, 52.3)
- moved C6 5.08 mm to (165.9, 47.0), turned to 0 degrees
- moved U3 4.50 mm to (140.4, 56.6)
- moved C1 4.26 mm to (165.8, 44.9)
- moved C5 4.24 mm to (165.8, 42.6), turned to 180 degrees
- moved R28 1.94 mm to (140.4, 62.3)
- moved R39 1.51 mm to (169.9, 95.1)
- moved Q4 1.45 mm to (170.1, 97.7)
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Connections:
- net /Sheet5FC7E9FD/CLK_25MHZ renamed /xc6slx16/CLK_25MHZ
- net /Sheet5FC7E9FD/DDR_VREF renamed /xc6slx16/DDR_VREF
- net /Sheet5FC7E9FD/FPGA_M0 renamed /xc6slx16/FPGA_M0
- net /Sheet5FC7E9FD/FPGA_M1 renamed /xc6slx16/FPGA_M1
- net /Sheet5FC7E9FD/HPD_EN renamed /hdmi-in/HPD_EN
- net /Sheet5FC7E9FD/HPD_NOTIFY renamed /hdmi-in/HPD_NOTIFY
- net /Sheet5FC7E9FD/QSPI_CLK renamed /xc6slx16/QSPI_CLK
- net /Sheet5FC7E9FD/QSPI_CS0 renamed /xc6slx16/QSPI_CS0
- net /Sheet5FC7E9FD/QSPI_DQ0 renamed /xc6slx16/QSPI_DQ0
- net /Sheet5FC7E9FD/QSPI_DQ1 renamed /xc6slx16/QSPI_DQ1
- net /Sheet5FC7E9FD/QSPI_DQ2 renamed /xc6slx16/QSPI_DQ2
- net /Sheet5FC7E9FD/QSPI_DQ3 renamed /xc6slx16/QSPI_DQ3
- net /Sheet5FC7E9FD/SCL renamed /hdmi-in/SCL
- net /Sheet5FC7E9FD/SDA renamed /hdmi-in/SDA
- net /Sheet5FC7E9FD/SDRAM_A0 renamed /lpddrsdram/SDRAM_A0
- net /Sheet5FC7E9FD/SDRAM_A1 renamed /lpddrsdram/SDRAM_A1
- net /Sheet5FC7E9FD/SDRAM_A10 renamed /lpddrsdram/SDRAM_A10
- net /Sheet5FC7E9FD/SDRAM_A11 renamed /lpddrsdram/SDRAM_A11
- net /Sheet5FC7E9FD/SDRAM_A12 renamed /lpddrsdram/SDRAM_A12
- net /Sheet5FC7E9FD/SDRAM_A13 renamed /lpddrsdram/SDRAM_A13
- net /Sheet5FC7E9FD/SDRAM_A14 renamed /xc6slx16/SDRAM_A14
- net /Sheet5FC7E9FD/SDRAM_A2 renamed /lpddrsdram/SDRAM_A2
- net /Sheet5FC7E9FD/SDRAM_A3 renamed /lpddrsdram/SDRAM_A3
- net /Sheet5FC7E9FD/SDRAM_A4 renamed /lpddrsdram/SDRAM_A4
- net /Sheet5FC7E9FD/SDRAM_A5 renamed /lpddrsdram/SDRAM_A5
- net /Sheet5FC7E9FD/SDRAM_A6 renamed /lpddrsdram/SDRAM_A6
- net /Sheet5FC7E9FD/SDRAM_A7 renamed /lpddrsdram/SDRAM_A7
- net /Sheet5FC7E9FD/SDRAM_A8 renamed /lpddrsdram/SDRAM_A8
- net /Sheet5FC7E9FD/SDRAM_A9 renamed /lpddrsdram/SDRAM_A9
- net /Sheet5FC7E9FD/SDRAM_BA0 renamed /lpddrsdram/SDRAM_BA0
- net /Sheet5FC7E9FD/SDRAM_BA1 renamed /lpddrsdram/SDRAM_BA1
- net /Sheet5FC7E9FD/SDRAM_CAS_N renamed /lpddrsdram/SDRAM_CAS_N
- net /Sheet5FC7E9FD/SDRAM_CKE renamed /lpddrsdram/SDRAM_CKE
- net /Sheet5FC7E9FD/SDRAM_CLK_N renamed /lpddrsdram/SDRAM_CLK_N
- net /Sheet5FC7E9FD/SDRAM_CLK_P renamed /lpddrsdram/SDRAM_CLK_P
- net /Sheet5FC7E9FD/SDRAM_CS_N renamed /lpddrsdram/SDRAM_CS_N
- net /Sheet5FC7E9FD/SDRAM_DQ0 renamed /lpddrsdram/SDRAM_DQ0
- net /Sheet5FC7E9FD/SDRAM_DQ1 renamed /lpddrsdram/SDRAM_DQ1
- net /Sheet5FC7E9FD/SDRAM_DQ10 renamed /lpddrsdram/SDRAM_DQ10
- net /Sheet5FC7E9FD/SDRAM_DQ11 renamed /lpddrsdram/SDRAM_DQ11
- net /Sheet5FC7E9FD/SDRAM_DQ12 renamed /lpddrsdram/SDRAM_DQ12
- net /Sheet5FC7E9FD/SDRAM_DQ13 renamed /lpddrsdram/SDRAM_DQ13
- net /Sheet5FC7E9FD/SDRAM_DQ14 renamed /lpddrsdram/SDRAM_DQ14
- net /Sheet5FC7E9FD/SDRAM_DQ15 renamed /lpddrsdram/SDRAM_DQ15
- net /Sheet5FC7E9FD/SDRAM_DQ2 renamed /lpddrsdram/SDRAM_DQ2
- net /Sheet5FC7E9FD/SDRAM_DQ3 renamed /lpddrsdram/SDRAM_DQ3
- net /Sheet5FC7E9FD/SDRAM_DQ4 renamed /lpddrsdram/SDRAM_DQ4
- net /Sheet5FC7E9FD/SDRAM_DQ5 renamed /lpddrsdram/SDRAM_DQ5
- net /Sheet5FC7E9FD/SDRAM_DQ6 renamed /lpddrsdram/SDRAM_DQ6
- net /Sheet5FC7E9FD/SDRAM_DQ7 renamed /lpddrsdram/SDRAM_DQ7
- net /Sheet5FC7E9FD/SDRAM_DQ8 renamed /lpddrsdram/SDRAM_DQ8
- net /Sheet5FC7E9FD/SDRAM_DQ9 renamed /lpddrsdram/SDRAM_DQ9
- net /Sheet5FC7E9FD/SDRAM_DQM0 renamed /lpddrsdram/SDRAM_DQM0
- net /Sheet5FC7E9FD/SDRAM_DQM1 renamed /lpddrsdram/SDRAM_DQM1
- net /Sheet5FC7E9FD/SDRAM_DQS0 renamed /lpddrsdram/SDRAM_DQS0
- net /Sheet5FC7E9FD/SDRAM_DQS1 renamed /lpddrsdram/SDRAM_DQS1
- net /Sheet5FC7E9FD/SDRAM_RAS_N renamed /lpddrsdram/SDRAM_RAS_N
- net /Sheet5FC7E9FD/SDRAM_WE_N renamed /lpddrsdram/SDRAM_WE_N
- net /Sheet5FC7E9FD/TMDS0_N renamed /hdmi-in/TMDS0_N
- net /Sheet5FC7E9FD/TMDS0_P renamed /hdmi-in/TMDS0_P
- net /Sheet5FC7E9FD/TMDS1_N renamed /hdmi-in/TMDS1_N
- net /Sheet5FC7E9FD/TMDS1_P renamed /hdmi-in/TMDS1_P
- net /Sheet5FC7E9FD/TMDS2_N renamed /hdmi-in/TMDS2_N
- net /Sheet5FC7E9FD/TMDS2_P renamed /hdmi-in/TMDS2_P
- net /Sheet5FC7E9FD/TMDS_CLK_N renamed /hdmi-in/TMDS_CLK_N
- net /Sheet5FC7E9FD/TMDS_CLK_P renamed /hdmi-in/TMDS_CLK_P
- IC4 pad 4: LCD_PWREN -> /power/LCD_PWREN
- IC5 pad 4: /Sheet5FC7E9FD/BL_DIM -> /power/BL_DIM
- R15 pad 1: LCD_PWREN -> /power/LCD_PWREN
- R70 pad 1: /Sheet5FC7E9FD/BL_DIM -> /power/BL_DIM
- U1 pad A4: Net-(U1-PadA4) -> /power/BL_DIM
- U1 pad A5: Net-(U1-PadA5) -> DBG_O1
- U1 pad A6: DBG_O2 -> DBG_O5
- U1 pad A7: Net-(U1-PadA7) -> DBG_O9
- U1 pad A9: LCD_PWREN -> Net-(U1-PadA9)
- U1 pad B5: Net-(U1-PadB5) -> DBG_O0
- U1 pad B6: DBG_O3 -> DBG_O4
- U1 pad C5: Net-(U1-PadC5) -> DBG_O3
- U1 pad C6: /Sheet5FC7E9FD/DBG_RX -> DBG_RX
- U1 pad C7: Net-(U1-PadC7) -> DBG_O8
- U1 pad C9: /Sheet5FC7E9FD/BL_DIM -> Net-(U1-PadC9)
- U1 pad D5: Net-(U1-PadD5) -> DBG_O2
- U1 pad D6: /Sheet6028E9E5/DBG_RX -> DBG_TX
- U1 pad E6: DBG_O0 -> DBG_O7
- U1 pad F7: DBG_O1 -> DBG_O6
- U1 pad N4: LCD_PWREN -> Net-(U1-PadN4)
- U1 pad T4: Net-(U1-PadT4) -> /power/LCD_PWREN
- U3 pad 8: /Sheet5FC7E9FD/DBG_RX -> DBG_TX
- U3 pad 9: /Sheet6028E9E5/DBG_RX -> DBG_RX
Routing:
- net +3V3: track 23.6 -> 350.6 mm, vias 8 -> 20
- net GND: track 57.2 -> 330.2 mm, vias 26 -> 56
- net V_DDR: track 29.2 -> 179.7 mm, vias 19 -> 21
- net +5V: track 0.00 -> 134.1 mm, vias 0 -> 7
- net +2V5: track 9.22 -> 95.0 mm, vias 8 -> 9
- net FPGA_TDO: track 0.71 -> 56.4 mm, vias 1 -> 3
- net +1V2: track 9.78 -> 62.7 mm, vias 8 -> 9
- net FPGA_TMS: track 0.00 -> 52.2 mm, vias 0 -> 1
- net FPGA_TCK: track 0.71 -> 51.2 mm, vias 1 -> 2
- net FPGA_TDI: track 0.71 -> 49.9 mm
- net LCD_BOOST_FB: track 10.7 -> 53.8 mm
- net DBG_TX: track 0.00 -> 36.6 mm, vias 0 -> 4
- net DBG_RX: track 0.00 -> 34.5 mm, vias 0 -> 4
- net DBG_O6: track 0.00 -> 33.3 mm, vias 0 -> 1
- net DBG_O7: track 0.00 -> 31.4 mm, vias 0 -> 1
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- added copper zone on L2, net GND
Other:
- board text added: "1"
- board text added: "2"
- board text added: "3"
- board text added: "4"
