File: xc6slx16-devboard-rev1/xc6slx16-devboard.kicad_pcb (KiCad board)
At the start: 4 copper layers, 75 x 65 mm, 141 parts, among them IC1 LM26480, IC2 M25P80-VMN6P, IC3 25MHz, IC4 SOT95P275X110-5N, IC5 SOT95P275X110-5N, J1 10118241-001RLF, J2 Conn_02x15_Odd_Even, J3 Conn_02x05_Odd_Even, J4 Conn_02x15_Odd_Even, J5 USB_C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

Commit message: sync rev1
Routing:
- net +1V2: track 62.7 -> 59.6 mm
- net V_DDR: track 179.7 -> 181.1 mm
- net FPGA_TDO: track 56.4 -> 55.7 mm
- net /lpddrsdram/SDRAM_DQ9: track 19.2 -> 18.5 mm
- net +3V3: track 350.6 -> 351.3 mm
Other:
- net class 2: via_dia 0.4 -> 0.45
- net class Default: via_dia 0.4 -> 0.45
- rule via_min_size: 0.4 -> 0.45
